File: js220_fp_template.kicad_pcb (KiCad board)
At the start: 2 copper layers, 95 x 24.7 mm, 5 parts, among them J1 JS220

Commit message: Update to use JS220 symbol and locked PCB items
Parts:
- TP1: value TestPoint -> Chassis Ground
Connections:
- net /I+ renamed I+
