File: js220_usbc.kicad_sch (KiCad schematic)
At the start: 14 parts, among them J1 JS220, J2 USB_C_Receptacle, J3 USB_C_Receptacle

Commit message: Fix polarity...
Connections:
- net VBUS_DEV: now also J1.3 (I-), J1.4 (I-); no longer J1.1 (I-), J1.2 (I-)
- net VBUS_SRC: now also J1.1 (I+), J1.2 (I+); no longer J1.3 (I+), J1.4 (I+)
Changed lines of the file:
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@@
   (title_block
     (title "Joulescope JS220 USB-C")
-    (date "2022-10-29")
-    (rev "1.0")
+    (date "2022-12-21")
+    (rev "1.1")
     (company "Alvaro Prieto")
   )

Commit message: v1.2 Done
Parts:
- added SW1: SW_DPDT_x2, snapeda:SW_JS202011SCQN, symbol Switch:SW_DPDT_x2
Connections:
- net CC1_DEV: now also SW1.4 (A); no longer C1.1
- net CC2_DEV: now also SW1.1 (A); no longer C2.1
- net RX1+: now also J3.A2 (TX1+); no longer J3.B11 (RX1+)
- net RX1-: now also J3.A3 (TX1-); no longer J3.B10 (RX1-)
- net RX2+: now also J3.B2 (TX2+); no longer J3.A11 (RX2+)
- net RX2-: now also J3.B3 (TX2-); no longer J3.A10 (RX2-)
- net SBU1: now also J3.B8 (SBU2); no longer J3.A8 (SBU1)
- net SBU2: now also J3.A8 (SBU1); no longer J3.B8 (SBU2)
- net TX1+: now also J3.B11 (RX1+); no longer J3.A2 (TX1+)
- net TX1-: now also J3.B10 (RX1-); no longer J3.A3 (TX1-)
- net TX2+: now also J3.A11 (RX2+); no longer J3.B2 (TX2+)
- net TX2-: now also J3.A10 (RX2-); no longer J3.B3 (TX2-)
- new net: C2.1, SW1.2 (B)
- new net: C1.1, SW1.5 (B)
- no-connect marks 0 -> 2
Other:
- note added: "Low-pass Filter to block USB-PD communications. Leaving USB-PD intact would mean VBUS voltages of up to 20V, which would be out of spec for the Joulescope. Use SW1 to restore USB-PD at your own risk!"
- note removed: "Low-pass Filter to block USB-PD communications. Leaving USB-PD intact would mean VBUS voltages of up to 20V, which would be out of spec for the Joulescope. Remove C1/C2 to restore USB-PD at your own risk!"
- moved on the sheet: C1, C2
